Commit message: update parcels size

File: belt_n_parcel_description/urdf/large_parcel.urdf (robot description, URDF)
Before this commit: robot large_parcel, 2 links, 1 joints
Links:
- added link large_parcel_3, mass 0.1; collision box size=0.25 0.25 0.01; visual box size=0.25 0.25 0.01
- link large_parcel_2: geometry collision box size=0.2 0.2 0.01; visual box size=0.2 0.2 0.01
Joints:
- removed joint large_parcel_joint
- added joint lower_parcel_joint: type fixed, parent large_parcel_1, child large_parcel_2, origin xyz=0.01 0.05 0.01 rpy=0.0 0.0 0.0, axis 0 0 0
- added joint upper_parcel_joint: type fixed, parent large_parcel_2, child large_parcel_3, origin xyz=0.05 0.05 0.01 rpy=0.0 0.0 0.0, axis 0 0 0

File: belt_n_parcel_description/urdf/medium_parcel.urdf (robot description, URDF)
Before this commit: robot medium_parcel, 2 links, 1 joints
Links:
- added link medium_parcel_3, mass 0.1; collision box size=0.1 0.1 0.003; visual box size=0.1 0.1 0.003
- link medium_parcel_1: geometry collision box size=0.1 0.1 0.008; visual box size=0.1 0.1 0.008
- link medium_parcel_2: geometry collision box size=0.1 0.1 0.005; visual box size=0.1 0.1 0.005
Joints:
- removed joint medium_parcel_joint
- added joint lower_parcel_joint: type fixed, parent medium_parcel_1, child medium_parcel_2, origin xyz=0.05 0.01 0.003 rpy=0.0 0.0 0.0, axis 0 0 0
- added joint upper_parcel_joint: type fixed, parent medium_parcel_2, child medium_parcel_3, origin xyz=-0.01 0.01 0.003 rpy=0.0 0.0 0.0, axis 0 0 0

File: belt_n_parcel_description/urdf/small_parcel.urdf (robot description, URDF)
Before this commit: robot small_parcel, 2 links, 1 joints
Links:
- added link small_parcel_3, mass 0.1; collision box size=0.015 0.015 0.003; visual box size=0.015 0.015 0.003
- link small_parcel_1: geometry collision box size=0.15 0.15 0.003; visual box size=0.1 0.1 0.003
- link small_parcel_2: geometry collision box size=0.15 0.15 0.003; visual box size=0.09 0.07 0.003
Joints:
- removed joint small_parcel_joint
- added joint lowerl_parcel_joint: type fixed, parent small_parcel_1, child small_parcel_2, origin xyz=0.01 0.01 0.003 rpy=0.0 0.0 0.0, axis 0 0 0
- added joint upper_parcel_joint: type fixed, parent small_parcel_2, child small_parcel_3, origin xyz=0.01 0.01 0.003 rpy=0.0 0.0 0.0, axis 0 0 0
